File: venusos_rpi_breakout.kicad_sch (KiCad schematic)
At the start: 48 parts, among them J1 8P8C, J10 RPi PWR, J11 5V+ Powersupply, J12 8P8C, J2 JST-MINI-4p, J3 JST-MINI-4p, J4 Screw Terminal, J5 Screw_Terminal_01x03, J6 Screw_Terminal_01x03, J7 Relay 1|2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

Commit message: Add files via upload
Other:
- note added: "Dual-SRD (12V)"
- note removed: "Dual-SRD (12V) - tbd"
Changed lines of the file:
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@@
     (effects (font (size 3 3)) (justify left bottom))
   )
-  (text "Dual-SRD (12V) - tbd" (at 15.24 69.85 0)
+  (text "Dual-SRD (12V)" (at 15.24 69.85 0)
     (effects (font (size 3 3)) (justify left bottom))
   )
